Commit message: remove unued files , add ui file , streamlit app , update files paths , add project plan , refactor code , separate simulation helper functions

File: assets/urdfs/pawn.urdf (robot description, URDF)
Before this commit: robot ChessPawn, 1 links, 0 joints
Links:
- link pawn_body: geometry collision cylinder length=0.05 radius=0.012; visual mesh filename=./meshes/Pawn.stl scale=0.003 0.003 0.003
