Commit message: update configration to support black and white colors

File: assets/urdfs/bishop.urdf (robot description, URDF)
Before this commit: robot ChessPawn, 1 links, 0 joints
Links:
- removed link pawn_body
- added link base_link, mass 0.04; collision cylinder length=0.05 radius=0.012; visual mesh filename=./meshes/Bishops.stl scale=0.003 0.003 0.003

File: assets/urdfs/bishop_b.urdf (robot description, URDF)
Before this commit: robot rook_w, 1 links, 0 joints
Links:
- link base_link: geometry collision cylinder length=0.05 radius=0.012; visual mesh filename=./meshes/Bishops.stl scale=0.003 0.003 0.003

File: assets/urdfs/king.urdf (robot description, URDF)
Before this commit: robot ChessPawn, 1 links, 0 joints
Links:
- removed link pawn_body
- added link base_link, mass 0.04; collision cylinder length=0.05 radius=0.012; visual mesh filename=./meshes/King.stl scale=0.003 0.003 0.003

File: assets/urdfs/king_b.urdf (robot description, URDF)
Before this commit: robot rook_w, 1 links, 0 joints
Links:
- link base_link: geometry collision cylinder length=0.05 radius=0.012; visual mesh filename=./meshes/King.stl scale=0.003 0.003 0.003

File: assets/urdfs/knight.urdf (robot description, URDF)
Before this commit: robot ChessPawn, 1 links, 0 joints
Links:
- removed link pawn_body
- added link base_link, mass 0.04; collision cylinder length=0.05 radius=0.012; visual mesh filename=./meshes/Knight.stl scale=0.003 0.003 0.003

File: assets/urdfs/knight_b.urdf (robot description, URDF)
Before this commit: robot rook_w, 1 links, 0 joints
Links:
- link base_link: geometry collision cylinder length=0.05 radius=0.012; visual mesh filename=./meshes/Knight.stl scale=0.003 0.003 0.003

File: assets/urdfs/pawn.urdf (robot description, URDF)
Before this commit: robot ChessPawn, 1 links, 0 joints
Links:
- removed link pawn_body
- added link base_link, mass 0.04; collision cylinder length=0.05 radius=0.012; visual mesh filename=./meshes/Pawn.stl scale=0.003 0.003 0.003

File: assets/urdfs/pawn_b.urdf (robot description, URDF)
Before this commit: robot rook_w, 1 links, 0 joints
Links:
- link base_link: geometry collision cylinder length=0.05 radius=0.012; visual mesh filename=./meshes/Pawn.stl scale=0.003 0.003 0.003

File: assets/urdfs/queen.urdf (robot description, URDF)
Before this commit: robot ChessPawn, 1 links, 0 joints
Links:
- removed link pawn_body
- added link base_link, mass 0.04; collision cylinder length=0.05 radius=0.012; visual mesh filename=./meshes/Queen.stl scale=0.003 0.003 0.003

File: assets/urdfs/queen_b.urdf (robot description, URDF)
Before this commit: robot rook_w, 1 links, 0 joints
Links:
- link base_link: geometry collision cylinder length=0.05 radius=0.012; visual mesh filename=./meshes/Queen.stl scale=0.003 0.003 0.003
